File: PCB/Sensor/Eagle/sensor_004.sch (EAGLE design)
At the start: 254 parts, among them IC1 LMV324, IC10 LMV324, IC11 LMV324, IC12 LMV324, IC13 LMV324, IC14 LMV324, IC15 LMV324, IC16 LMV324, IC17 LMV324, IC18 LMV324, IC19 LMV324, IC2 LMV324, IC20 LMV324, IC21 LMV324, IC22 LMV324, IC23 LMV324, IC24 LMV324, IC3 LMV324, IC4 LMV324, IC5 LMV324, IC6 LMV324, IC7 LMV324, IC8 LMV324, IC9 LMV324, U1 74HC4067, U2 74HC4067, U3 74HC4067, U4 74HC4067, U5 74HC4067, U6 74HC4067

Commit message: change sensor board and case
Parts:
- PHD1, PHD10, PHD11, PHD12, PHD13, PHD14, PHD15, PHD16, PHD17, PHD18, PHD19, PHD2, PHD20, PHD21, PHD22, PHD23, PHD24, PHD25, PHD26, PHD27, PHD28, PHD29, PHD3, PHD30, PHD31, PHD32, PHD33, PHD34, PHD35, PHD36, PHD37, PHD38, PHD39, PHD4, PHD40, PHD41, PHD42, PHD43, PHD44, PHD45, PHD46, PHD47, PHD48, PHD49, PHD5, PHD50, PHD51, PHD52, PHD53, PHD54, PHD55, PHD56, PHD57, PHD58, PHD59, PHD6, PHD60, PHD61, PHD62, PHD63, PHD64, PHD65, PHD66, PHD67, PHD68, PHD69, PHD7, PHD70, PHD71, PHD72, PHD73, PHD74, PHD75, PHD76, PHD77, PHD78, PHD79, PHD8, PHD80, PHD81, PHD82, PHD83, PHD84, PHD85, PHD86, PHD87, PHD88, PHD89, PHD9, PHD90, PHD91, PHD92, PHD93, PHD94, PHD95, PHD96: device Miroculus:PD_0.2 -> Miroculus:PD_2
Connections:
- net +5V: now also J2.6; no longer J2.5
- net GND: now also J2.5; no longer J2.6
